File: PCB/5Vto-2V5.kicad_sch (KiCad schematic)
At the start: 3 parts, among them U8 TPS72325DBVT

Commit message: more footprints
Parts:
- C24: footprint (none) -> Capacitor_SMD:C_1210_3225Metric_Pad1.33x2.70mm_HandSolder
Changed lines of the file:
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@@
 			)
 		)
-		(property "Footprint" ""
+		(property "Footprint" "Capacitor_SMD:C_1210_3225Metric_Pad1.33x2.70mm_HandSolder"
 			(at 171.7548 97.79 0)
 			(effects

Commit message: cap footprints finished
Parts:
- C23: footprint (none) -> Capacitor_SMD:C_0201_0603Metric_Pad0.64x0.40mm_HandSolder
Changed lines of the file:
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@@
 			)
 		)
-		(property "Footprint" ""
+		(property "Footprint" "Capacitor_SMD:C_0201_0603Metric_Pad0.64x0.40mm_HandSolder"
 			(at 134.9248 99.06 0)
 			(effects

Commit message: initial pcb import
Parts:
- U8: footprint TPS72325DBVT:SOT95P280X145-5N -> CustomLib:72325
Changed lines of the file:
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@@
 			)
 		)
-		(property "Footprint" "TPS72325DBVT:SOT95P280X145-5N"
+		(property "Footprint" "CustomLib:72325"
 			(at 160.02 104.14 0)
 			(effects
