File: PCB/ADS1299.kicad_sch (KiCad schematic)
At the start: 0 parts

Commit message: RP2040 sheet
Parts:
- added C1: 1.5nF, symbol Device:C
- added C10, C14, C16, C2, C4, C8: 0.1µF, symbol Device:C
- added C11, C12, C15, C17, C5, C6, C9: 1µF, symbol Device:C
- added C13: 100µF, symbol Device:C
- added C3: 10µF, symbol Device:C
- added C7: 1nF, symbol Device:C
- added CN1, CN2, CN3, CN4: W2A41C681KAT2A, W2A41C681KAT2A:CAPCAXE50P210X130X94-8N, symbol custom_lib:W2A41C681KAT2A
- added R1: 1MΩ, symbol Device:R
- added R2: 20kΩ, symbol Device:R
- added R3, R6, R7, R8, R9: 10kΩ, symbol Device:R
- added RN1, RN2, RN3, RN4: CAY16-103J4LF, CAY16-103J4LF:RESCAF80P320X160X60-8N, symbol custom_lib:CAY16-103J4LF
- added U1: ADS1299IPAGR, PAG64_TEX, symbol ads199:ADS1299IPAGR
- added U3, U4, U9: TPD4E1B06DCKR, TPD4E1B06DCKR:SOT65P210X110-6N, symbol custom_lib:TPD4E1B06DCKR
Connections:
- new net: C2.2, C3.1, U1.24 (VREFP)
- new net: R9.1, U1.46 (GPIO4)
- new net: C13.1, U1.28 (VCAP1)
- new net: R7.1, U1.44 (GPIO2)
- new net: C8.2, C9.2, U1.55 (VCAP3)
- new net: R6.2, U1.52 (CLKSEL)
- new net: R3.1, U1.42 (GPIO1)
- new net: C12.1, U1.30 (VCAP2)
- new net: C1.1, R1.1, U1.61 (BIASINV)
- new net: R8.1, U1.45 (GPIO3)
- new net: C5.1, U1.26 (VCAP4)
- new net +2V5: C10.2, C11.2, C14.1, C15.1, U1.19 (AVDD), U1.21 (AVDD), U1.22 (AVDD), U1.54 (AVDD1), U1.56 (AVDD), U1.59 (AVDD)
- new net +3V3: C16.1, C17.1, R6.1, U1.48 (DVDD), U1.50 (DVDD)
- new net -2V5: C10.1, C11.1, C12.2, C13.2, C2.1, C3.2, C4.1, C5.2, C6.1, C8.1, C9.1, U1.17 (SRB1), U1.18 (SRB2), U1.20 (AVSS), U1.23 (AVSS), U1.25 (VREFN), U1.32 (AVSS), U1.53 (AVSS1), U1.57 (AVSS), U1.58 (AVSS), U1.60 (BIASREF)
- new net Bias: C1.2, C7.2, R1.2, R2.1, U1.62 (BIASIN), U1.63 (BIASOUT)
- new net GND: C14.2, C15.2, C16.2, C17.2, C4.2, C6.2, C7.1, CN1.5, CN1.6, CN1.7, CN1.8, CN2.5, CN2.6, CN2.7, CN2.8, CN3.5, CN3.6, CN3.7, CN3.8, CN4.5, CN4.6, CN4.7, CN4.8, R3.2, R7.2, R8.2, R9.2, U1.31 (RESV1), U1.33 (DGND), U1.41 (DAISY_IN), U1.49 (DGND), U1.51 (DGND), U1.64 (RESERVED), U3.3 (GND), U4.3 (GND), U9.2 (IO2), U9.3 (GND), U9.4 (IO3), U9.5 (IO4)
- new net I1: RN4.2, RN4.3, U3.2 (IO2)
- new net I2: RN3.4, RN4.1, U3.4 (IO3)
- new net I3: RN3.2, RN3.3, U3.5 (IO4)
- new net I4: RN2.4, RN3.1, U4.1 (IO1)
- new net I5: RN2.2, RN2.3, U4.2 (IO2)
- new net I6: RN1.4, RN2.1, U4.4 (IO3)
- new net I7: RN1.2, RN1.3, U4.5 (IO4)
- new net I8: RN1.1, RN4.4, U3.1 (IO1)
- new net IB: R2.2, U9.1 (IO1)
- new net IN1N: CN4.4, RN4.5, U1.15 (IN1N)
- new net IN1P: CN4.3, RN4.6, U1.16 (IN1P)
- new net IN2N: CN4.2, RN4.7, U1.13 (IN2N)
- new net IN2P: CN4.1, RN4.8, U1.14 (IN2P)
- new net IN3N: CN3.4, RN3.5, U1.11 (IN3N)
- new net IN3P: CN3.3, RN3.6, U1.12 (IN3P)
- new net IN4N: CN3.2, RN3.7, U1.9 (IN4N)
- new net IN4P: CN3.1, RN3.8, U1.10 (IN4P)
- new net IN5N: CN2.4, RN2.5, U1.7 (IN5N)
- new net IN5P: CN2.3, RN2.6, U1.8 (IN5P)
- new net IN6N: CN2.2, RN2.7, U1.5 (IN6N)
- new net IN6P: CN2.1, RN2.8, U1.6 (IN6P)
- new net IN7N: CN1.4, RN1.5, U1.3 (IN7N)
- new net IN7P: CN1.3, RN1.6, U1.4 (IN7P)
- new net IN8N: CN1.2, RN1.7, U1.1 (IN8N)
- new net IN8P: CN1.1, RN1.8, U1.2 (IN8P)
Other:
- note added: "1nF"
- note added: "20kΩ"

Commit message: ads1299 sheet
Parts:
- removed CN1, CN3, CN4: W2A41C681KAT2A, W2A41C681KAT2A:CAPCAXE50P210X130X94-8N, symbol custom_lib:W2A41C681KAT2A
- removed RN1, RN2, RN3, RN4: CAY16-103J4LF, CAY16-103J4LF:RESCAF80P320X160X60-8N, symbol custom_lib:CAY16-103J4LF
- added CN5, CN6, CN7: W2A41C681KAT2A, W2A41C681KAT2A:CAPCAXE50P210X130X94-8N, symbol custom_lib:W2A41C681KAT2A
- added RN5, RN6, RN7, RN8: CAY16-103J4LF, CAY16-103J4LF:RESCAF80P320X160X60-8N, symbol custom_lib:CAY16-103J4LF
- C10, C14, C4: value 0.1µF -> 1µF
- C11, C15, C6: value 1µF -> 0.1µF
Connections:
- net IB is gone; now on net Bias: R2.2, U9.1 (IO1)
- net +2V5: now also C10.1, C11.1, C4.1, C6.1; no longer C10.2, C11.2, C14.1, C15.1
- net -2V5: now also C10.2, C11.2, C14.1, C15.1; no longer C10.1, C11.1, C4.1, C6.1
- net Bias: now also C7.1; no longer C7.2
- net GND: now also C7.2, CN2.1, CN2.2, CN2.3, CN2.4, CN5.1, CN5.2, CN5.3, CN5.4, CN6.1, CN6.2, CN6.3, CN6.4, CN7.1, CN7.2, CN7.3, CN7.4; no longer C7.1, CN2.5, CN2.6, CN2.7, CN2.8
- net I1: now also RN8.2, RN8.3
- net I2: now also RN7.4, RN8.1
- net I3: now also RN7.2, RN7.3
- net I4: now also RN6.4, RN7.1
- net I5: now also RN6.2, RN6.3
- net I6: now also RN5.4, RN6.1
- net I7: now also RN5.2, RN5.3
- net I8: now also RN5.1, RN8.4
- net IN1N: now also CN7.8, RN8.5
- net IN1P: now also CN7.7, RN8.6
- net IN2N: now also CN7.6, RN8.7
- net IN2P: now also CN7.5, RN8.8
- net IN3N: now also CN6.8, RN7.5
- net IN3P: now also CN6.7, RN7.6
- net IN4N: now also CN6.6, RN7.7
- net IN4P: now also CN6.5, RN7.8
- net IN5N: now also CN5.8, RN6.5; no longer CN2.4
- net IN5P: now also CN5.7, RN6.6; no longer CN2.3
- net IN6N: now also CN5.6, RN6.7; no longer CN2.2
- net IN6P: now also CN5.5, RN6.8; no longer CN2.1
- net IN7N: now also CN2.8, RN5.5
- net IN7P: now also CN2.7, RN5.6
- net IN8N: now also CN2.6, RN5.7
- net IN8P: now also CN2.5, RN5.8
- net MOSI: now reaches U1.34 (DIN)
- net PDWN: now reaches U1.35 (*PWDN)
- net RESET: now reaches U1.36 (*RESET)
- net START: now reaches U1.38 (START)
- net CS: now reaches U1.39 (*CS)
- net SCLK: now reaches U1.40 (SCLK)
- net MISO: now reaches U1.43 (DOUT)
- net DRDY: now reaches U1.47 (*DRDY)
Other:
- note added: "ADS1299"
- note added: "Bias Input Module"
- note added: "Bypass Capacitors"
- note added: "ESD Module"
- note added: "Input Module 1"
- note added: "Input Module 2"
- note added: "Input Module 3"
- note added: "Input Module 4"
- moved on the sheet: C1, C12, C13, C2, C3, C5, C8, C9, R1, R3, R6, R7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
