File: PCB/ADS1299.kicad_sch (KiCad schematic)
At the start: 37 parts, among them CN2 W2A41C681KAT2A, CN5 W2A41C681KAT2A, CN6 W2A41C681KAT2A, CN7 W2A41C681KAT2A, U1 ADS1299IPAGR, U3 TPD4E1B06DCKR, U4 TPD4E1B06DCKR, U9 TPD4E1B06DCKR

Commit message: v0.1, pre-grounding
Parts:
- removed CN2, CN5, CN6, CN7: W2A41C681KAT2A, CustomLib:W3A41C102MAT2A, symbol custom_lib:W2A41C681KAT2A
- added C25, C26, C31, C32, C33, C34, C35, C36, C37, C38, C39, C40, C41, C42, C43, C44: 1nF, Capacitor_SMD:C_0603_1608Metric_Pad1.08x0.95mm_HandSolder, symbol Device:C
Connections:
- net GND: now also C25.2, C26.2, C31.2, C32.2, C33.2, C34.2, C35.2, C36.2, C37.2, C38.2, C39.2, C40.2, C41.2, C42.2, C43.2, C44.2
- net I1: now also RN5.1, RN8.4, U3.1 (IO1); no longer RN8.2, RN8.3, U3.2 (IO2)
- net I2: now also RN8.2, RN8.3, U3.2 (IO2); no longer RN7.4, RN8.1, U3.4 (IO3)
- net I3: now also RN7.4, RN8.1, U3.4 (IO3); no longer RN7.2, RN7.3, U3.5 (IO4)
- net I4: now also RN7.2, RN7.3, U3.5 (IO4); no longer RN6.4, RN7.1, U4.1 (IO1)
- net I5: now also RN6.4, RN7.1, U4.1 (IO1); no longer RN6.2, RN6.3, U4.2 (IO2)
- net I6: now also RN6.2, RN6.3, U4.2 (IO2); no longer RN5.4, RN6.1, U4.4 (IO3)
- net I7: now also RN5.4, RN6.1, U4.4 (IO3); no longer RN5.2, RN5.3, U4.5 (IO4)
- net I8: now also RN5.2, RN5.3, U4.5 (IO4); no longer RN5.1, RN8.4, U3.1 (IO1)
- net IN1N: now also RN8.6, C26.1; no longer RN8.5
- net IN1P: now also RN8.5, C25.1; no longer RN8.6
- net IN2N: now also RN8.8, C32.1; no longer RN8.7
- net IN2P: now also RN8.7, C31.1; no longer RN8.8
- net IN3N: now also RN7.6, C34.1; no longer RN7.5
- net IN3P: now also RN7.5, C33.1; no longer RN7.6
- net IN4N: now also RN7.8, C36.1; no longer RN7.7
- net IN4P: now also RN7.7, C35.1; no longer RN7.8
- net IN5N: now also RN6.6, C38.1; no longer RN6.5
- net IN5P: now also RN6.5, C37.1; no longer RN6.6
- net IN6N: now also RN6.8, C40.1; no longer RN6.7
- net IN6P: now also RN6.7, C39.1; no longer RN6.8
- net IN7N: now also RN5.6, C42.1; no longer RN5.5
- net IN7P: now also RN5.5, C41.1; no longer RN5.6
- net IN8N: now also RN5.8, C44.1; no longer RN5.7
- net IN8P: now also RN5.7, C43.1; no longer RN5.8
Other:
- note removed: "1nF"
