File: PCB/5Vto-5V.kicad_sch (KiCad schematic)
At the start: 3 parts, among them U5 LM2664M6

Commit message: start of footprints
Parts:
- C18, C22: value 3.3µF -> 10µF
Changed lines of the file:
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@@
 			)
 		)
-		(property "Value" "3.3µF "
+		(property "Value" "10µF "
 			(at 167.386 111.252 0)
 			(effects
@@
 			)
 		)
-		(property "Value" "3.3µF "
+		(property "Value" "10µF "
 			(at 125.476 110.744 0)
 			(effects

Commit message: more footprints
Parts:
- C18, C22: footprint (none) -> Capacitor_SMD:C_0805_2012Metric_Pad1.18x1.45mm_HandSolder
Changed lines of the file:
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@@
 			)
 		)
-		(property "Footprint" ""
+		(property "Footprint" "Capacitor_SMD:C_0805_2012Metric_Pad1.18x1.45mm_HandSolder"
 			(at 171.7548 106.68 0)
 			(effects
@@
 			)
 		)
-		(property "Footprint" ""
+		(property "Footprint" "Capacitor_SMD:C_0805_2012Metric_Pad1.18x1.45mm_HandSolder"
 			(at 129.8448 106.68 0)
 			(effects

Commit message: initial pcb import
Parts:
- U5: footprint LM2664M6:SOT95P300X120-6N -> CustomLib:lm266
Changed lines of the file:
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@@
 			)
 		)
-		(property "Footprint" "LM2664M6:SOT95P300X120-6N"
+		(property "Footprint" "CustomLib:lm266"
 			(at 156.21 107.95 0)
 			(effects
