File: PCB/5Vto2V5.kicad_sch (KiCad schematic)
At the start: 3 parts, among them U11 TPS73225DBVR

Commit message: start of footprints
Parts:
- C29: footprint (none) -> Capacitor_SMD:C_0402_1005Metric_Pad0.74x0.62mm_HandSolder
Changed lines of the file:
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@@
 			)
 		)
-		(property "Footprint" ""
+		(property "Footprint" "Capacitor_SMD:C_0402_1005Metric_Pad0.74x0.62mm_HandSolder"
 			(at 129.8448 101.6 0)
 			(effects

Commit message: cap footprints finished
Parts:
- C30: footprint (none) -> Capacitor_SMD:C_0201_0603Metric_Pad0.64x0.40mm_HandSolder
Changed lines of the file:
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@@
 			)
 		)
-		(property "Footprint" ""
+		(property "Footprint" "Capacitor_SMD:C_0201_0603Metric_Pad0.64x0.40mm_HandSolder"
 			(at 142.5448 101.6 0)
 			(effects

Commit message: initial pcb import
Parts:
- U11: footprint TPS73225DBVR:SOT95P280X145-5N -> CustomLib:73225
Changed lines of the file:
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@@
 			)
 		)
-		(property "Footprint" "TPS73225DBVR:SOT95P280X145-5N"
+		(property "Footprint" "CustomLib:73225"
 			(at 167.64 106.68 0)
 			(effects
