File: PCB/5Vto3V3.kicad_sch (KiCad schematic)
At the start: 3 parts, among them U7 TPS73233DBVT

Commit message: start of footprints
Parts:
- C27: footprint (none) -> Capacitor_SMD:C_0402_1005Metric_Pad0.74x0.62mm_HandSolder
Changed lines of the file:
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@@
 			)
 		)
-		(property "Footprint" ""
+		(property "Footprint" "Capacitor_SMD:C_0402_1005Metric_Pad0.74x0.62mm_HandSolder"
 			(at 133.6548 104.14 0)
 			(effects

Commit message: cap footprints finished
Parts:
- C28: footprint (none) -> Capacitor_SMD:C_0201_0603Metric_Pad0.64x0.40mm_HandSolder
Changed lines of the file:
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@@
 			)
 		)
-		(property "Footprint" ""
+		(property "Footprint" "Capacitor_SMD:C_0201_0603Metric_Pad0.64x0.40mm_HandSolder"
 			(at 146.3548 104.14 0)
 			(effects

Commit message: initial pcb import
Parts:
- U7: footprint TPS73233DBVT:SOT95P280X145-5N -> CustomLib:73233
Changed lines of the file:
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@@
 			)
 		)
-		(property "Footprint" "TPS73233DBVT:SOT95P280X145-5N"
+		(property "Footprint" "CustomLib:73233"
 			(at 171.45 109.22 0)
 			(effects
