File: PCB/power.kicad_sch (KiCad schematic)
At the start: 7 parts, among them U6 TPS61023DRLR

Commit message: start of footprints
Parts:
- C20, C21: footprint (none) -> Capacitor_SMD:C_1210_3225Metric_Pad1.33x2.70mm_HandSolder
- L1: footprint (none) -> CustomLib:IND_74438357010_WRE
- U6: footprint DRL0006A -> (none)
Changed lines of the file:
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@@
 			)
 		)
-		(property "Footprint" ""
+		(property "Footprint" "Capacitor_SMD:C_1210_3225Metric_Pad1.33x2.70mm_HandSolder"
 			(at 169.2148 102.87 0)
 			(effects
@@
 			)
 		)
-		(property "Footprint" ""
+		(property "Footprint" "CustomLib:IND_74438357010_WRE"
 			(at 140.97 87.63 0)
 			(effects
@@
 			)
 		)
-		(property "Footprint" "DRL0006A"
+		(property "Footprint" ""
 			(at 148.59 99.06 0)
 			(effects
@@
 			)
 		)
-		(property "Footprint" ""
+		(property "Footprint" "Capacitor_SMD:C_1210_3225Metric_Pad1.33x2.70mm_HandSolder"
 			(at 180.6448 102.87 0)
 			(effects

Commit message: more footprints
Parts:
- C19: footprint (none) -> Capacitor_SMD:C_0805_2012Metric_Pad1.18x1.45mm_HandSolder
Changed lines of the file:
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@@
 			)
 		)
-		(property "Footprint" ""
+		(property "Footprint" "Capacitor_SMD:C_0805_2012Metric_Pad1.18x1.45mm_HandSolder"
 			(at 121.6152 102.87 0)
 			(effects

Commit message: res footprints
Parts:
- R4, R5: footprint (none) -> Resistor_SMD:R_0805_2012Metric_Pad1.20x1.40mm_HandSolder
Changed lines of the file:
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@@
 			)
 		)
-		(property "Footprint" ""
+		(property "Footprint" "Resistor_SMD:R_0805_2012Metric_Pad1.20x1.40mm_HandSolder"
 			(at 154.432 110.49 90)
 			(effects
@@
 			)
 		)
-		(property "Footprint" ""
+		(property "Footprint" "Resistor_SMD:R_0805_2012Metric_Pad1.20x1.40mm_HandSolder"
 			(at 154.432 102.87 90)
 			(effects

Commit message: final footprints
Parts:
- U6: footprint (none) -> CustomLib:SOTFL50P160X60-6N
Changed lines of the file:
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@@
 			)
 		)
-		(property "Footprint" ""
+		(property "Footprint" "CustomLib:SOTFL50P160X60-6N"
 			(at 148.59 99.06 0)
 			(effects
