File: v2/v2.kicad_pcb (KiCad board)
At the start: 4 copper layers, 45.5 x 52 mm, 60 parts, among them CN1 W2A41C681KAT2A, CN2 W2A41C681KAT2A, CN3 W2A41C681KAT2A, CN4 W2A41C681KAT2A, J1 Conn_01x02_Pin, J2 Conn_01x09_Pin, J3 Conn_01x20_Socket, J4 Conn_01x20_Socket, U1 ADS1299IPAGR, U11 TPS73225DBVR, U3 TPD4E1B06DCKR, U4 TPD4E1B06DCKR, U5 LM2664M6, U6 TPS61023DRLR, U7 TPS73233DBVT, U8 TPS72325DBVT, U9 TPD4E1B06DCKR

Commit message: test pins
Parts:
- added J5: Conn_01x01_Pin, Connector_PinHeader_2.54mm:PinHeader_1x01_P2.54mm_Vertical, F.Cu at (143.9, 73.3)
- added J6: Conn_01x01_Pin, Connector_PinHeader_2.54mm:PinHeader_1x01_P2.54mm_Vertical, F.Cu at (147.4, 99.4)
- added J7: Conn_01x01_Pin, Connector_PinHeader_2.54mm:PinHeader_1x01_P2.54mm_Vertical, F.Cu at (127.3, 83.8)
- added J8: Conn_01x01_Pin, Connector_PinHeader_2.54mm:PinHeader_1x01_P2.54mm_Vertical, F.Cu at (131.1, 97.9)
Connections:
- J2 pad 1: /ADS1299/Bias -> /ADS1299/BI
- R2 pad 2: /ADS1299/Bias -> /ADS1299/BI
- U9 pad 1: /ADS1299/Bias -> /ADS1299/BI
Routing:
- net GND: track 74.9 -> 87.4 mm, vias 37 -> 51
- net +2V5: track 38.9 -> 47.4 mm
- net -2V5: track 44.3 -> 52.5 mm, vias 8 -> 11
- net /ADS1299/Bias: track 17.9 -> 9.84 mm, vias 1 -> 0
- net /ADS1299/BI: track 0.00 -> 8.09 mm, vias 0 -> 1
- net +3V3: track 20.5 -> 24.4 mm
- net +5V: track 91.1 -> 93.5 mm

Commit message: final v02
Parts:
- moved J6 20.3 mm to (127.1, 98.7)
- moved J8 4.88 mm to (127.1, 95.1)
- moved C1 3.39 mm to (131.4, 96.9), turned to -90 degrees
- moved R1 1.60 mm to (129.9, 96.9), turned to -90 degrees
Routing:
- net GND: track 87.4 -> 95.9 mm, vias 51 -> 52
- net -2V5: track 52.5 -> 48.8 mm, vias 11 -> 12
- net /ADS1299/Bias: track 9.84 -> 7.65 mm
- net Net-(U1-BIASIN): track 3.75 -> 4.87 mm
- net /ADS1299/START: track 41.3 -> 42.3 mm
Other:
- board text added: "+2V5"
- board text added: "+3V3"
- board text added: "+5V"
- board text added: "-2V5"
- board text added: "BATTERY USE ONLY OR"
- board text added: "RISK ELECTROCUTION"
- board text removed: "BATTERY USE ONLY OR RISK ELECTROCUTION"
