File: v2/5Vto-2V5.kicad_sch (KiCad schematic)
At the start: 3 parts, among them U8 TPS72325DBVT

Commit message: footprint reset for v0.2
Parts:
- C23: footprint Capacitor_SMD:C_0201_0603Metric_Pad0.64x0.40mm_HandSolder -> (none)
- C24: footprint Capacitor_SMD:C_1210_3225Metric_Pad1.33x2.70mm_HandSolder -> (none)
Changed lines of the file:
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@@
 			)
 		)
-		(property "Footprint" "Capacitor_SMD:C_1210_3225Metric_Pad1.33x2.70mm_HandSolder"
+		(property "Footprint" ""
 			(at 171.7548 97.79 0)
 			(effects
@@
 			)
 		)
-		(property "Footprint" "Capacitor_SMD:C_0201_0603Metric_Pad0.64x0.40mm_HandSolder"
+		(property "Footprint" ""
 			(at 134.9248 99.06 0)
 			(effects

Commit message: new footprints
Parts:
- C23, C24: footprint (none) -> Capacitor_SMD:C_0603_1608Metric_Pad1.08x0.95mm_HandSolder
Changed lines of the file:
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@@
 			)
 		)
-		(property "Footprint" ""
+		(property "Footprint" "Capacitor_SMD:C_0603_1608Metric_Pad1.08x0.95mm_HandSolder"
 			(at 171.7548 97.79 0)
 			(effects
@@
 			)
 		)
-		(property "Footprint" ""
+		(property "Footprint" "Capacitor_SMD:C_0603_1608Metric_Pad1.08x0.95mm_HandSolder"
 			(at 134.9248 99.06 0)
 			(effects

Commit message: v2 code
Parts:
- C23: value 0.01µF -> 0.01µF
- C24: value 22µF -> 22µF
Changed lines of the file:
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@@
 			)
 		)
-		(property "Value" "22µF "
+		(property "Value" "22µF"
 			(at 167.894 102.362 0)
 			(effects
@@
 			)
 		)
-		(property "Value" "0.01µF "
+		(property "Value" "0.01µF"
 			(at 130.81 103.378 0)
 			(effects
