File: v2/5Vto-5V.kicad_sch (KiCad schematic)
At the start: 3 parts, among them U5 LM2664M6

Commit message: footprint reset for v0.2
Parts:
- C18, C22: footprint Capacitor_SMD:C_0805_2012Metric_Pad1.18x1.45mm_HandSolder -> (none)
Changed lines of the file:
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@@
 			)
 		)
-		(property "Footprint" "Capacitor_SMD:C_0805_2012Metric_Pad1.18x1.45mm_HandSolder"
+		(property "Footprint" ""
 			(at 171.7548 106.68 0)
 			(effects
@@
 			)
 		)
-		(property "Footprint" "Capacitor_SMD:C_0805_2012Metric_Pad1.18x1.45mm_HandSolder"
+		(property "Footprint" ""
 			(at 129.8448 106.68 0)
 			(effects

Commit message: new footprints
Parts:
- C18, C22: footprint (none) -> Capacitor_SMD:C_0603_1608Metric_Pad1.08x0.95mm_HandSolder
Changed lines of the file:
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@@
 			)
 		)
-		(property "Footprint" ""
+		(property "Footprint" "Capacitor_SMD:C_0603_1608Metric_Pad1.08x0.95mm_HandSolder"
 			(at 171.7548 106.68 0)
 			(effects
@@
 			)
 		)
-		(property "Footprint" ""
+		(property "Footprint" "Capacitor_SMD:C_0603_1608Metric_Pad1.08x0.95mm_HandSolder"
 			(at 129.8448 106.68 0)
 			(effects

Commit message: v2 code
Parts:
- C18, C22: value 10µF -> 10µF
Changed lines of the file:
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@@
 			)
 		)
-		(property "Value" "10µF "
+		(property "Value" "10µF"
 			(at 167.386 111.252 0)
 			(effects
@@
 			)
 		)
-		(property "Value" "10µF "
+		(property "Value" "10µF"
 			(at 125.476 110.744 0)
 			(effects
