File: v2/5Vto2V5.kicad_sch (KiCad schematic)
At the start: 3 parts, among them U11 TPS73225DBVR

Commit message: footprint reset for v0.2
Parts:
- C29: footprint Capacitor_SMD:C_0402_1005Metric_Pad0.74x0.62mm_HandSolder -> (none)
- C30: footprint Capacitor_SMD:C_0201_0603Metric_Pad0.64x0.40mm_HandSolder -> (none)
Changed lines of the file:
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@@
 			)
 		)
-		(property "Footprint" "Capacitor_SMD:C_0402_1005Metric_Pad0.74x0.62mm_HandSolder"
+		(property "Footprint" ""
 			(at 129.8448 101.6 0)
 			(effects
@@
 			)
 		)
-		(property "Footprint" "Capacitor_SMD:C_0201_0603Metric_Pad0.64x0.40mm_HandSolder"
+		(property "Footprint" ""
 			(at 142.5448 101.6 0)
 			(effects

Commit message: new footprints
Parts:
- C29, C30: footprint (none) -> Capacitor_SMD:C_0603_1608Metric_Pad1.08x0.95mm_HandSolder
Changed lines of the file:
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@@
 			)
 		)
-		(property "Footprint" ""
+		(property "Footprint" "Capacitor_SMD:C_0603_1608Metric_Pad1.08x0.95mm_HandSolder"
 			(at 129.8448 101.6 0)
 			(effects
@@
 			)
 		)
-		(property "Footprint" ""
+		(property "Footprint" "Capacitor_SMD:C_0603_1608Metric_Pad1.08x0.95mm_HandSolder"
 			(at 142.5448 101.6 0)
 			(effects

Commit message: v2 code
Parts:
- C29: value 1µF -> 1µF
- C30: value 0.01µF -> 0.01µF
Changed lines of the file:
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@@
 			)
 		)
-		(property "Value" "1µF "
+		(property "Value" "1µF"
 			(at 125.984 106.172 0)
 			(effects
@@
 			)
 		)
-		(property "Value" "0.01µF "
+		(property "Value" "0.01µF"
 			(at 138.43 105.918 0)
 			(effects
