File: v2/5Vto3V3.kicad_sch (KiCad schematic)
At the start: 3 parts, among them U7 TPS73233DBVT

Commit message: footprint reset for v0.2
Parts:
- C27: footprint Capacitor_SMD:C_0402_1005Metric_Pad0.74x0.62mm_HandSolder -> (none)
- C28: footprint Capacitor_SMD:C_0201_0603Metric_Pad0.64x0.40mm_HandSolder -> (none)
Changed lines of the file:
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@@
 			)
 		)
-		(property "Footprint" "Capacitor_SMD:C_0402_1005Metric_Pad0.74x0.62mm_HandSolder"
+		(property "Footprint" ""
 			(at 133.6548 104.14 0)
 			(effects
@@
 			)
 		)
-		(property "Footprint" "Capacitor_SMD:C_0201_0603Metric_Pad0.64x0.40mm_HandSolder"
+		(property "Footprint" ""
 			(at 146.3548 104.14 0)
 			(effects

Commit message: new footprints
Parts:
- C27, C28: footprint (none) -> Capacitor_SMD:C_0603_1608Metric_Pad1.08x0.95mm_HandSolder
Changed lines of the file:
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@@
 			)
 		)
-		(property "Footprint" ""
+		(property "Footprint" "Capacitor_SMD:C_0603_1608Metric_Pad1.08x0.95mm_HandSolder"
 			(at 133.6548 104.14 0)
 			(effects
@@
 			)
 		)
-		(property "Footprint" ""
+		(property "Footprint" "Capacitor_SMD:C_0603_1608Metric_Pad1.08x0.95mm_HandSolder"
 			(at 146.3548 104.14 0)
 			(effects

Commit message: v2 code
Parts:
- C27: value 1µF -> 1µF
- C28: value 0.01µF -> 0.01µF
Changed lines of the file:
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@@
 			)
 		)
-		(property "Value" "1µF "
+		(property "Value" "1µF"
 			(at 129.794 108.712 0)
 			(effects
@@
 			)
 		)
-		(property "Value" "0.01µF "
+		(property "Value" "0.01µF"
 			(at 142.24 108.458 0)
 			(effects
