File: v2/v2.kicad_sch (KiCad schematic)
At the start: 2 parts, among them J1 Conn_01x02_Pin, J2 Conn_01x09_Pin

Commit message: test pins
Parts:
- added J5, J6, J7, J8: Conn_01x01_Pin, Connector_PinHeader_2.54mm:PinHeader_1x01_P2.54mm_Vertical, symbol Connector:Conn_01x01_Pin
Connections:
- net +2V5: now also J8.1 (Pin_1)
- net +3V3: now also J7.1 (Pin_1)
- net +5V: now also J5.1 (Pin_1)
- net -2V5: now also J6.1 (Pin_1)
- net ADS1299/Bias renamed ADS1299/BI
Other:
- sheet ADS1299 ports: added BI; removed Bias

Commit message: v2 code
Other:
- moved on the sheet: J2
